File: hardware/kicad/controller_node/controller_node.kicad_sch (KiCad schematic)
At the start: 2 parts, among them U1 STM32F401RETx, U2 ER_OLEDM0.96_1x-I2C

Commit message: Update controller node project in Kicad
Parts:
- added J1: Jack-DC, symbol Connector:Jack-DC
- added M1, M2: Motor_Servo, symbol Motor:Motor_Servo
- added U3: HC-05, symbol New_Library:HC-05
Connections:
- net GND: now reaches U1.12 (VSSA)
- net GND: now also U1.18 (VSS), U1.31 (VSS), U1.47 (VSS), U1.63 (VSS), U2.1 (GND), J1.2, M1.3 (-), M2.3 (-), U3.3 (GND)
- net at U1.55 (PB3): now also M2.1 (PWM)
- net at U1.56 (PB4): now also M1.1 (PWM)
- net at U1.61 (PB8): now also U2.3 (SCL)
- net at U1.62 (PB9): now also U2.4 (SDA)
- new net: J1.1, M1.2 (+), M2.2 (+)

Commit message: Completed controller node schmeatic
Connections:
- net +5V: now reaches U3.2 (VCC)
- net at U3.4 (TXD): now also U1.43 (PA10)
- net at U3.6 (STATE): now also U1.9 (PC1)
- net at U1.42 (PA9): now also U3.4 (TXD)
- net +3.3V: now reaches U2.2 (VCC)
- no-connect marks 0 -> 2
